Commit message: 还是不行

File: fishbot_description/urdf/fishbot/actuator/wheel.urdf.xacro (robot description, xacro)
@@ -30,4 +30,6 @@
             <origin xyz="${xyz}" />
             <axis xyz="0 1 0" />
+            <limit effort="100.0" velocity="100.0"/>
+            <dynamics damping="0.01" friction="0.01"/>
         </joint>
     </xacro:macro>

File: fishbot_description/urdf/fishbot/fishbot.ros2_control.xacro (robot description, xacro)
@@ -11,8 +11,8 @@
                     <param name="max">100</param>
                 </command_interface>
-                <command_interface name="effort">
+                <!-- <command_interface name="effort">
                     <param name="min">-10</param>
                     <param name="max">10</param>
-                </command_interface>
+                </command_interface> -->
                 <state_interface name="position" />
                 <state_interface name="velocity" />
@@ -24,8 +24,8 @@
                     <param name="max">100</param>
                 </command_interface>
-                <command_interface name="effort">
+                <!-- <command_interface name="effort">
                     <param name="min">-10</param>
                     <param name="max">10</param>
-                </command_interface>
+                </command_interface> -->
                 <state_interface name="position" />
                 <state_interface name="velocity" />
